File: HW/rbpi-z-hat/rbpi-z-hat.kicad_pcb (KiCad board)
At the start: 4 copper layers, 65 x 30 mm, 94 parts, among them IC1 BQ24315DSGR, J1 RBPI_CONN, J10 JST_GH, J2 Conn_01x10, J3 Conn_01x10, J4 Conn_01x10, J5 Conn_01x06, J6 Conn_01x06, J7 Conn_01x06, J8 Conn_01x06_MountingPin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

Commit message: Routing
Parts:
- moved U3 0.23 mm to (49.2, 16.6)
Connections:
- net /rbpi/GPIO_4 renamed /rbpi/Pin_7_PPM_SBUS_INPUT
- net Net-(J3-Pad1) renamed /PCA9685/SERVO_POWER
- IC1 pad 3: (no net) -> unconnected-(IC1-NC-Pad3)
- IC1 pad 4: (no net) -> /BQ24313/BQ_nFAULT
- J1 pad 11: (no net) -> /rbpi/Pin_11_UART_RTS
- J1 pad 12: (no net) -> /rbpi/Pin_12_UART_CTS
- J1 pad 13: (no net) -> /rbpi/Pin_13_PWM_EN
- J1 pad 15: (no net) -> /rbpi/GPIO_22
- J1 pad 16: (no net) -> /rbpi/Pin_16_MPU_DRDY
- J1 pad 18: (no net) -> /rbpi/Pin_18
- J1 pad 22: (no net) -> /rbpi/Pin_22
- J1 pad 24: /rbpi/SPI0_CE0 -> /LSM_nCS
- J1 pad 26: /rbpi/SPI0_CE1 -> /BMP_nCS
- J1 pad 27: (no net) -> /rbpi/GPIO_0_HAT_SDA
- J1 pad 28: (no net) -> /rbpi/GPIO_1_HAT_SCL
- J1 pad 29: (no net) -> /rbpi/GPIO_5
- J1 pad 31: (no net) -> /rbpi/GPIO_6
- J1 pad 32: (no net) -> /rbpi/GPIO_12
- J1 pad 33: (no net) -> /rbpi/GPIO_13
- J1 pad 35: (no net) -> /rbpi/GPIO_19
- J1 pad 36: (no net) -> /rbpi/Pin_36
- J1 pad 37: (no net) -> /rbpi/GPIO_26
- J1 pad 38: (no net) -> /rbpi/Pin_38
- J1 pad 40: (no net) -> /rbpi/Pin_40
- L8 pad 1: (no net) -> /FB/Y4
- L8 pad 2: (no net) -> /FB/X4
- R11 pad 2: /rbpi/SPI0_CE1 -> /BMP_nCS
- RN6 pad 4: (no net) -> unconnected-(RN6-R4.1-Pad4)
- RN6 pad 6: (no net) -> /rbpi/SBUS_INPUT_RAW
- RN7 pad 4: /rbpi/SPI0_CE0 -> /LSM_nCS
- U1 pad 3: (no net) -> /SENSORS_EN
- U1 pad 4: (no net) -> unconnected-(U1-NC-Pad4)
- U5 pad 2: (no net) -> /BMP_nCS
- U6 pad 2: (no net) -> unconnected-(U6-ALERT/RDY-Pad2)
- U6 pad 6: (no net) -> /ADS1015/AIN2
- U6 pad 7: (no net) -> /ADS1015/AIN3
- U8 pad 10: (no net) -> /IMU/LSM_INT3
- U8 pad 11: (no net) -> /IMU/LSM_INT1
- U8 pad 12: (no net) -> /IMU/LSM_INT2
- U8 pad 13: (no net) -> /IMU/LSM_DEN
- U8 pad 7: /IMU/LSM_nCS -> /LSM_nCS
- U8 pad 8: /IMU/LSM_nCS -> /LSM_nCS
- U8 pad 9: (no net) -> /IMU/LSM_INT4
- U9 pad 10: Net-(U9-Pad10) -> unconnected-(U9-RESV-Pad10)
- U9 pad 11: Net-(U9-Pad10) -> unconnected-(U9-RESV-Pad11)
- U9 pad 12: (no net) -> /IMU/ICM_nCS
- U9 pad 2: Net-(U9-Pad10) -> unconnected-(U9-RESV-Pad2)
- U9 pad 3: Net-(U9-Pad10) -> unconnected-(U9-RESV-Pad3)
- U9 pad 4: (no net) -> /IMU/ICM_INT1
- U9 pad 7: Net-(U9-Pad10) -> unconnected-(U9-RESV-Pad7)
- U9 pad 9: (no net) -> /IMU/ICM_INT2
- X1 pad 1: (no net) -> unconnected-(X1-EN-Pad1)
Routing:
- net /SCL1: track 0.00 -> 44.1 mm, vias 0 -> 1
- net /SDA1: track 0.00 -> 42.2 mm, vias 0 -> 1
- net /PCA9685/PWM_OUT0: track 0.00 -> 14.7 mm, vias 0 -> 1
- net /PCA9685/PWM_OUT1: track 0.00 -> 13.3 mm, vias 0 -> 1
- net /PCA9685/PWM_OUT2: track 0.00 -> 12.0 mm, vias 0 -> 1
- net /PCA9685/PWM_OUT3: track 0.00 -> 10.9 mm, vias 0 -> 1
- net /PCA9685/PCA_VDD: track 0.00 -> 6.54 mm
- net /PCA9685/PWM_OUT10: track 0.00 -> 5.68 mm, vias 0 -> 1
- net /PCA9685/PWM_OUT9: track 0.00 -> 5.38 mm, vias 0 -> 1
- net /PCA9685/PWM_OUT8: track 0.00 -> 4.93 mm, vias 0 -> 1
- net /PCA9685/PWM_0: track 0.00 -> 4.57 mm
- net /PCA9685/PWM_10: track 0.00 -> 4.39 mm
- net /PCA9685/PWM_4: track 0.00 -> 4.37 mm
- net /PCA9685/PWM_7: track 0.00 -> 4.31 mm
- net /PCA9685/PWM_3: track 0.00 -> 4.18 mm
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